File: JFET_Preamp_Daughter/daughter.kicad_pcb (KiCad board)
At the start: 2 copper layers, 50 x 40 mm, 21 parts, among them J101 Conn_01x08_Socket, J102 Conn_01x06, J103 Conn_01x06, U101 PCM1865DBTR

Commit message: generate gerber and drill files
Other:
- board text removed: "5/3/2026"
- board text removed: "JFET Preamp with ADC Daughterboard By Lucas Samaniego"
Changed lines of the file:
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@@
 			(plot_on_all_layers_selection 0x00000000_00000000_00000000_00000000)
 			(disableapertmacros no)
-			(usegerberextensions no)
+			(usegerberextensions yes)
 			(usegerberattributes yes)
 			(usegerberadvancedattributes yes)
@@
 			(outputformat 1)
 			(mirror no)
-			(drillshape 1)
+			(drillshape 0)
 			(scaleselection 1)
-			(outputdirectory "")
+			(outputdirectory "Gerber_Plot_6-30-2026/")
 		)
 	)
@@
 		)
 	)
-	(gr_text "JFET Preamp with ADC Daughterboard				By Lucas Samaniego"
-		(at 102.25 128 0)
-		(layer "F.SilkS")
-		(effects
-			(font
-				(size 1 1)
-				(thickness 0.1)
-			)
-			(justify left bottom)
-		)
-	)
-	(gr_text "5/3/2026"
-		(at 119.75 131.75 0)
-		(layer "F.SilkS")
-		(effects
-			(font
-				(size 1 1)
-				(thickness 0.1)
-			)
-			(justify left bottom)
-		)
-	)
 	(gr_text "COMM\nSTATUS"
 		(at 56.25 35.25 0)
@@
 	)
 	(segment
-		(start 56.35 27)
-		(end 56.35 28.4)
-		(width 0.2)
-		(layer "F.Cu")
-		(net "/CH3_COLD")
-	)
-	(segment
-		(start 56.35 28.4)
-		(end 48 36.75)
-		(width 0.2)
-		(layer "F.Cu")
-		(net "/CH3_COLD")
-	)
-	(segment
-		(start 48 36.75)
-		(end 48 39.5)
-		(width 0.2)
-		(layer "F.Cu")
-		(net "/CH3_COLD")
-	)
-	(segment
-		(start 53.81 27)
-		(end 53.81 28.44)
-		(width 0.2)
-		(layer "F.Cu")
-		(net "/CH4_COLD")
-	)
-	(segment
-		(start 53.81 28.44)
-		(end 47 35.25)
-		(width 0.2)
-		(layer "F.Cu")
-		(net "/CH4_COLD")
-	)
-	(segment
-		(start 47 35.25)
-		(end 47 39.18)
-		(width 0.2)
-		(layer "F.Cu")
-		(net "/CH4_COLD")
-	)
-	(segment
-		(start 46.19 28.31)
-		(end 46 28.5)
-		(width 0.2)
-		(layer "F.Cu")
-		(net "/CH3_HOT")
-	)
-	(segment
-		(start 46 28.5)
-		(end 46 39.18)
-		(width 0.2)
-		(layer "F.Cu")
-		(net "/CH3_HOT")
-	)
-	(segment
-		(start 46.19 27)
-		(end 46.19 28.31)
-		(width 0.2)
-		(layer "F.Cu")
-		(net "/CH3_HOT")
-	)
-	(segment
-		(start 43.65 27)
-		(end 45 28.35)
-		(width 0.2)
-		(layer "F.Cu")
-		(net "/CH4_HOT")
-	)
-	(segment
-		(start 45 28.35)
-		(end 45 39.18)
-		(width 0.2)
-		(layer "F.Cu")
-		(net "/CH4_HOT")
-	)
-	(segment
 		(start 46.5 61.25)
 		(end 46.5 50.82)
@@
 	)
 	(segment
-		(start 53.81 61.56)
-		(end 47.5 55.25)
+		(start 56.35 27)
+		(end 56.35 28.4)
 		(width 0.2)
 		(layer "F.Cu")
-		(net "/CH1_HOT")
+		(net "/CH3_COLD")
 	)
 	(segment
-		(start 47.5 55.25)
-		(end 47.5 50.32)
+		(start 56.35 28.4)
+		(end 48 36.75)
 		(width 0.2)
 		(layer "F.Cu")
-		(net "/CH1_HOT")
+		(net "/CH3_COLD")
 	)
 	(segment
-		(start 53.81 63)
-		(end 53.81 61.56)
+		(start 48 36.75)
+		(end 48 39.5)
 		(width 0.2)
 		(layer "F.Cu")
-		(net "/CH1_HOT")
+		(net "/CH3_COLD")
+	)
+	(segment
+		(start 46.19 28.31)
+		(end 46 28.5)
+		(width 0.2)
+		(layer "F.Cu")
+		(net "/CH3_HOT")
+	)
+	(segment
+		(start 46 28.5)
+		(end 46 39.18)
+		(width 0.2)
+		(layer "F.Cu")
+		(net "/CH3_HOT")
+	)
+	(segment
+		(start 46.19 27)
+		(end 46.19 28.31)
+		(width 0.2)
+		(layer "F.Cu")
+		(net "/CH3_HOT")
 	)
 	(segment
@@
 		(net "/CH2_HOT")
 	)
+	(segment
+		(start 43.65 27)
+		(end 45 28.35)
+		(width 0.2)
+		(layer "F.Cu")
+		(net "/CH4_HOT")
+	)
+	(segment
+		(start 45 28.35)
+		(end 45 39.18)
+		(width 0.2)
+		(layer "F.Cu")
+		(net "/CH4_HOT")
+	)
+	(segment
+		(start 53.81 61.56)
+		(end 47.5 55.25)
+		(width 0.2)
+		(layer "F.Cu")
+		(net "/CH1_HOT")
+	)
+	(segment
+		(start 47.5 55.25)
+		(end 47.5 50.32)
+		(width 0.2)
+		(layer "F.Cu")
+		(net "/CH1_HOT")
+	)
+	(segment
+		(start 53.81 63)
+		(end 53.81 61.56)
+		(width 0.2)
+		(layer "F.Cu")
+		(net "/CH1_HOT")
+	)
+	(segment
+		(start 53.81 27)
+		(end 53.81 28.44)
+		(width 0.2)
+		(layer "F.Cu")
+		(net "/CH4_COLD")
+	)
+	(segment
+		(start 53.81 28.44)
+		(end 47 35.25)
+		(width 0.2)
+		(layer "F.Cu")
+		(net "/CH4_COLD")
+	)
+	(segment
+		(start 47 35.25)
+		(end 47 39.18)
+		(width 0.2)
+		(layer "F.Cu")
+		(net "/CH4_COLD")
+	)
 	(zone
