File: JFET_Preamp_Mother/mother.kicad_pcb (KiCad board)
At the start: 2 copper layers, 140 x 120 mm, 102 parts, among them J101 Conn_01x02, J102 Conn_01x06_Socket, J103 Conn_01x06_Socket, J201 XLR3, J301 XLR3, J401 XLR3, J501 XLR3, Q101 AO3401A, Q201 2SK209, Q202 2SK209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

Commit message: regenerate mother gerber and drill
Other:
- board text removed: "5/3/2026"
- board text removed: "JFET Preamp with ADC Motherboard By Lucas Samaniego"
Changed lines of the file:
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@@
 			(outputformat 1)
 			(mirror no)
-			(drillshape 1)
+			(drillshape 0)
 			(scaleselection 1)
-			(outputdirectory "")
+			(outputdirectory "Gerber_Plot_6-30-2026/")
 		)
 	)
@@
 		(layer "Edge.Cuts")
 	)
-	(gr_text "5/3/2026"
-		(at 206.25 194 0)
-		(layer "F.Cu")
-		(effects
-			(font
-				(size 1.5 1.5)
-				(thickness 0.3)
-				(bold yes)
-			)
-			(justify left bottom)
-		)
-	)
 	(gr_text "PWR STATUS\n"
 		(at 106.5 34.5 0)
 		(layer "F.SilkS")
 		(effects
-			(font
-				(size 1 1)
-				(thickness 0.1)
-			)
-			(justify left bottom)
-		)
-	)
-	(gr_text "JFET Preamp with ADC Motherboard					By Lucas Samaniego"
-		(at 190 190 0)
-		(layer "F.SilkS")
-		(effects
