File: JFET_Preamp_Mother/mother.kicad_pcb (KiCad board)
At the start: 2 copper layers, 140 x 120 mm, 102 parts, among them J101 Conn_01x02, J102 Conn_01x06_Socket, J103 Conn_01x06_Socket, J201 XLR3, J301 XLR3, J401 XLR3, J501 XLR3, Q101 AO3401A, Q201 2SK209, Q202 2SK209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

Commit message: fixed TVS Diodes across 4 channels and redo placement and traces
Parts:
- D201, D202, D301, D302, D401, D402, D501, D502: footprint Package_TO_SOT_SMD:SOT-23 -> Diode_SMD:D_SMA
- moved D502 4.88 mm to (50.0, 24.5), turned to 90 degrees
- moved D402 4.83 mm to (50.0, 54.0), turned to 90 degrees
- moved D202 4.49 mm to (49.5, 114.2), turned to 90 degrees
- moved D302 4.17 mm to (49.8, 84.8), turned to 90 degrees
- moved R211 2.95 mm to (45.3, 116.8)
- moved R311 2.89 mm to (45.6, 86.8)
- moved R511 2.85 mm to (45.8, 27.0)
- moved R411 2.76 mm to (45.8, 57.0)
- moved D501 2.64 mm to (51.0, 38.8), turned to 90 degrees
- moved D201 2.46 mm to (50.5, 126.8), turned to 90 degrees
- moved D401 1.99 mm to (51.5, 66.5), turned to 90 degrees
- moved D301 1.80 mm to (51.5, 96.2), turned to 90 degrees
Routing:
- net /CH1_GND: track 123.2 -> 126.6 mm
- net Net-(D202-A2): track 57.0 -> 60.0 mm
- net Net-(D402-A2): track 58.5 -> 61.4 mm
- net /Channel_1/D_TVS_COLD: track 12.3 -> 9.80 mm
- net /Channel_2/D_TVS_COLD: track 12.3 -> 9.85 mm
- net /Channel_3/D_TVS_COLD: track 12.3 -> 10.0 mm
- net Net-(D502-A2): track 60.0 -> 62.1 mm
- net Net-(D302-A2): track 58.7 -> 60.8 mm
- net /Channel_4/D_TVS_COLD: track 12.3 -> 10.4 mm
- net /CH4_GND: track 110.8 -> 112.5 mm
- net /Channel_3/D_TVS_HOT: track 17.7 -> 16.5 mm
- net /Channel_2/D_TVS_HOT: track 17.7 -> 17.1 mm
- net /Channel_4/D_TVS_HOT: track 17.7 -> 18.2 mm
