File: JFET_Preamp_Mother/mother.kicad_sch (KiCad schematic)
At the start: 6 parts, among them J101 Conn_01x02

Commit message: motherboard .sch erc clean
Parts:
- added D101: BZV55C27, Diode_SMD:D_MiniMELF, symbol Diode:BZV55C27
- added D102: SMAJ26A, Diode_SMD:D_SMA, symbol Diode:SMAJ26A
- added F101: 0.5, downloaded_footprints:FUSRB510W51L790T310H1370, symbol Device:Polyfuse
- added J102, J103: Conn_01x06_Socket, symbol Connector:Conn_01x06_Socket
- added Q101: AO3401A, Package_TO_SOT_SMD:SOT-23, symbol Transistor_FET:AO3401A
- added R102: 4.7k, symbol Device:R
- R101: value 4.7k -> 100k; footprint Resistor_SMD:R_0603_1608Metric -> (none)
- renumbered D101 to D103
Connections:
- net +24V: now also R101.1, D102.2 (A2), Q101.3 (D), R102.2; no longer J101.1 (Pin_1), R101.2
- net CH1_COLD: now also J103.1 (Pin_1)
- net CH1_GND: now also J103.4 (Pin_4)
- net CH1_HOT: now also J103.5 (Pin_5)
- net CH2_COLD: now also J103.2 (Pin_2)
- net CH2_GND: now also J103.3 (Pin_3)
- net CH2_HOT: now also J103.6 (Pin_6)
- net CH3_COLD: now also J102.1 (Pin_1)
- net CH3_GND: now also J102.3 (Pin_3)
- net CH3_HOT: now also J102.5 (Pin_5)
- net CH4_COLD: now also J102.2 (Pin_2)
- net CH4_GND: now also J102.4 (Pin_4)
- net CH4_HOT: now also J102.6 (Pin_6)
- net GND: now also D101.1 (K), D102.1 (A1)
- net at D103.2 (A): now also R102.1; no longer R101.1
- new net: D101.2 (A), Q101.1 (G), R101.2
- new net: F101.1, Q101.2 (S)
- new net: F101.2, J101.1 (Pin_1)
Other:
- moved on the sheet: C101, C102, C103, D103, J101

Commit message: finish draft of mother/daughter sch and start routing, reconcile libraries and missing footprints
Parts:
- added R102: 0, symbol Device:R
- renumbered R102 to R103
Connections:
- net +24V: now also R102.1; no longer C101.1, C102.1, C103.1, D102.2 (A2), Q101.3 (D), R101.1, R103.2
- new net: C101.1, C102.1, C103.1, D102.2 (A2), Q101.3 (D), R101.1, R102.2, R103.2
Changed lines of the file:
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@@
+	)
+	(junction
+		(at 157.48 39.37)
+		(diameter 0)
+		(color 0 0 0 0)
+	)
+	(junction
+		(at 148.59 30.48)
+		(diameter 0)
+		(color 0 0 0 0)
+	)
+	(junction
+		(at 121.92 30.48)
+		(diameter 0)
+		(color 0 0 0 0)
+	)
+	(junction
+		(at 172.72 33.02)
+		(diameter 0)
+		(color 0 0 0 0)
+	)
+	(junction
+		(at 119.38 40.64)
+		(diameter 0)
+		(color 0 0 0 0)
+	)
+	(junction
+		(at 129.54 30.48)
+		(diameter 0)
+		(color 0 0 0 0)
+	)
+	(junction
+		(at 109.22 40.64)
+		(diameter 0)
+		(color 0 0 0 0)
 	)
 	(junction
@@
 	)
 	(junction
-		(at 157.48 39.37)
-		(diameter 0)
-		(color 0 0 0 0)
-	)
-	(junction
-		(at 148.59 30.48)
-		(diameter 0)
-		(color 0 0 0 0)
-	)
-	(junction
-		(at 121.92 30.48)
-		(diameter 0)
-		(color 0 0 0 0)
-	)
-	(junction
-		(at 172.72 33.02)
-		(diameter 0)
-		(color 0 0 0 0)
-	)
-	(junction
-		(at 119.38 40.64)
-		(diameter 0)
-		(color 0 0 0 0)
-	)
-	(junction
-		(at 129.54 30.48)
-		(diameter 0)
-		(color 0 0 0 0)
-	)
-	(junction
-		(at 109.22 40.64)
-		(diameter 0)
-		(color 0 0 0 0)
-	)
-	(junction
 		(at 119.38 30.48)
 		(diameter 0)
@@
 		(pts
 			(xy 173.99 27.94) (xy 173.99 30.48)
+		)
+		(stroke
+			(width 0)
+			(type default)
+		)
+	)
+	(wire
+		(pts
+			(xy 114.3 20.32) (xy 114.3 21.59)
 		)
 		(stroke
@@
 	)
 	(symbol
+		(lib_id "Device:R")
+		(at 114.3 25.4 0)
+		(unit 1)
+		(body_style 1)
+		(exclude_from_sim no)
+		(in_bom yes)
+		(on_board yes)
+		(in_pos_files yes)
+		(dnp no)
+		(property "Reference" "R102"
+			(at 115.824 24.384 0)
+			(show_name no)
+			(do_not_autoplace no)
+			(effects
+				(font
+					(size 1.27 1.27)
+				)
+				(justify left)
+			)
+		)
+		(property "Value" "0"
+			(at 115.824 26.162 0)
+			(show_name no)
+			(do_not_autoplace no)
+			(effects
+				(font
+					(size 1.27 1.27)
+				)
+				(justify left)
+			)
+		)
+		(property "Footprint" ""
+			(at 112.522 25.4 90)
+			(hide yes)
+			(show_name no)
+			(do_not_autoplace no)
+			(effects
+				(font
+					(size 1.27 1.27)
+				)
+			)
+		)
+		(property "Datasheet" ""
+			(at 114.3 25.4 0)
+			(hide yes)
+			(show_name no)
+			(do_not_autoplace no)
+			(effects
+				(font
+					(size 1.27 1.27)
+				)
+			)
+		)
+		(property "Description" "Resistor"
+			(at 114.3 25.4 0)
+			(hide yes)
+			(show_name no)
+			(do_not_autoplace no)
+			(effects
+				(font
+					(size 1.27 1.27)
+				)
+			)
+		)
+		(pin "2"
+		)
+		(pin "1"
+		)
+		(instances
+			(project "mother"
+				(path "/7a893922-4a26-4218-912f-8bb60bebfa2a"
+					(reference "R102")
+					(unit 1)
+				)
+			)
+		)
+	)
+	(symbol
 		(lib_id "power:PWR_FLAG")
 		(at 121.92 29.21 0)
@@
 		(in_pos_files yes)
 		(dnp no)
-		(property "Reference" "R102"
+		(property "Reference" "R103"
 			(at 104.14 26.162 90)
 			(show_name no)
@@
 			(project "mother"
 				(path "/7a893922-4a26-4218-912f-8bb60bebfa2a"
-					(reference "R102")
+					(reference "R103")
 					(unit 1)
 				)
@@
 	(symbol
 		(lib_id "power:+24V")
-		(at 114.3 29.21 0)
+		(at 114.3 20.32 0)
 		(unit 1)
 		(body_style 1)
@@
 		(dnp no)
 		(property "Reference" "#PWR0101"
-			(at 114.3 33.02 0)
+			(at 114.3 24.13 0)
 			(hide yes)
 			(show_name no)
@@
 		)
 		(property "Value" "+24V"
-			(at 114.3 25.4 0)
+			(at 114.3 16.51 0)
 			(show_name no)
 			(do_not_autoplace no)
@@
 		)
 		(property "Footprint" ""
-			(at 114.3 29.21 0)
+			(at 114.3 20.32 0)
 			(hide yes)
 			(show_name no)
@@
 		)
 		(property "Datasheet" ""
-			(at 114.3 29.21 0)
+			(at 114.3 20.32 0)
 			(hide yes)
 			(show_name no)
@@
 		)
 		(property "Description" "Power symbol creates a global label with name \"+24V\""
-			(at 114.3 29.21 0)
-			(hide yes)
-			(show_name no)
+			(at 114.3 20.32 0)
+			(hide yes)
+			(show_name no)

Commit message: forgot to save ERC change adding pwr flag to mother sch
Parts:
- J102, J103: footprint (none) -> Connector_PinSocket_2.54mm:PinSocket_1x06_P2.54mm_Vertical
- R101, R102, R103: footprint (none) -> Resistor_SMD:R_0603_1608Metric
Changed lines of the file:
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@@
+	)
+	(junction
+		(at 114.3 20.32)
+		(diameter 0)
+		(color 0 0 0 0)
 	)
 	(junction
@@
 	(wire
 		(pts
+			(xy 114.3 19.05) (xy 114.3 20.32)
+		)
+		(stroke
+			(width 0)
+			(type default)
+		)
+	)
+	(wire
+		(pts
+			(xy 114.3 29.21) (xy 114.3 30.48)
+		)
+		(stroke
+			(width 0)
+			(type default)
+		)
+	)
+	(wire
+		(pts
+			(xy 129.54 30.48) (xy 144.78 30.48)
+		)
+		(stroke
+			(width 0)
+			(type default)
+		)
+	)
+	(wire
+		(pts
+			(xy 100.33 43.18) (xy 109.22 43.18)
+		)
+		(stroke
+			(width 0)
+			(type default)
+		)
+	)
+	(wire
+		(pts
+			(xy 100.33 40.64) (xy 100.33 43.18)
+		)
+		(stroke
+			(width 0)
+			(type default)
+		)
+	)
+	(wire
+		(pts
+			(xy 129.54 41.91) (xy 144.78 41.91)
+		)
+		(stroke
+			(width 0)
+			(type default)
+		)
+	)
+	(wire
+		(pts
+			(xy 144.78 39.37) (xy 144.78 41.91)
+		)
+		(stroke
+			(width 0)
+			(type default)
+		)
+	)
+	(wire
+		(pts
+			(xy 162.56 33.02) (xy 162.56 46.99)
+		)
+		(stroke
+			(width 0)
+			(type default)
+		)
+	)
+	(wire
+		(pts
+			(xy 69.85 68.58) (xy 69.85 58.42)
+		)
+		(stroke
+			(width 0)
+			(type default)
+		)
+	)
+	(wire
+		(pts
 			(xy 114.3 20.32) (xy 114.3 21.59)
-		)
-		(stroke
-			(width 0)
-			(type default)
-		)
-	)
-	(wire
-		(pts
-			(xy 114.3 29.21) (xy 114.3 30.48)
-		)
-		(stroke
-			(width 0)
-			(type default)
-		)
-	)
-	(wire
-		(pts
-			(xy 129.54 30.48) (xy 144.78 30.48)
-		)
-		(stroke
-			(width 0)
-			(type default)
-		)
-	)
-	(wire
-		(pts
-			(xy 100.33 43.18) (xy 109.22 43.18)
-		)
-		(stroke
-			(width 0)
-			(type default)
-		)
-	)
-	(wire
-		(pts
-			(xy 100.33 40.64) (xy 100.33 43.18)
-		)
-		(stroke
-			(width 0)
-			(type default)
-		)
-	)
-	(wire
-		(pts
-			(xy 129.54 41.91) (xy 144.78 41.91)
-		)
-		(stroke
-			(width 0)
-			(type default)
-		)
-	)
-	(wire
-		(pts
-			(xy 144.78 39.37) (xy 144.78 41.91)
-		)
-		(stroke
-			(width 0)
-			(type default)
-		)
-	)
-	(wire
-		(pts
-			(xy 162.56 33.02) (xy 162.56 46.99)
-		)
-		(stroke
-			(width 0)
-			(type default)
-		)
-	)
-	(wire
-		(pts
-			(xy 69.85 68.58) (xy 69.85 58.42)
 		)
 		(stroke
@@
 			)
 		)
-		(property "Footprint" ""
+		(property "Footprint" "Resistor_SMD:R_0603_1608Metric"
 			(at 146.812 35.56 90)
 			(hide yes)
@@
 			)
 		)
-		(property "Footprint" ""
+		(property "Footprint" "Resistor_SMD:R_0603_1608Metric"
 			(at 112.522 25.4 90)
 			(hide yes)
@@
 			)
 		)
-		(property "Footprint" ""
+		(property "Footprint" "Resistor_SMD:R_0603_1608Metric"
 			(at 104.14 32.258 90)
 			(hide yes)
@@
 			)
 		)
-		(property "Footprint" ""
+		(property "Footprint" "Connector_PinSocket_2.54mm:PinSocket_1x06_P2.54mm_Vertical"
 			(at 74.93 53.34 0)
 			(hide yes)
@@
 	(symbol
 		(lib_id "power:+24V")
-		(at 114.3 20.32 0)
+		(at 114.3 19.05 0)
 		(unit 1)
 		(body_style 1)
@@
 		(dnp no)
 		(property "Reference" "#PWR0101"
-			(at 114.3 24.13 0)
+			(at 114.3 22.86 0)
 			(hide yes)
 			(show_name no)
@@
 		)
 		(property "Value" "+24V"
-			(at 114.3 16.51 0)
+			(at 114.3 15.24 0)
 			(show_name no)
 			(do_not_autoplace no)
@@
 		)
 		(property "Footprint" ""
-			(at 114.3 20.32 0)
+			(at 114.3 19.05 0)
 			(hide yes)
 			(show_name no)
@@
 		)
 		(property "Datasheet" ""
-			(at 114.3 20.32 0)
+			(at 114.3 19.05 0)
 			(hide yes)
 			(show_name no)
@@
 		)
 		(property "Description" "Power symbol creates a global label with name \"+24V\""
-			(at 114.3 20.32 0)
+			(at 114.3 19.05 0)
 			(hide yes)
 			(show_name no)
@@
 				(path "/7a893922-4a26-4218-912f-8bb60bebfa2a"
 					(reference "C102")
+					(unit 1)
+				)
+			)
+		)
+	)
+	(symbol
+		(lib_id "power:PWR_FLAG")
+		(at 114.3 20.32 90)
+		(unit 1)
+		(body_style 1)
+		(exclude_from_sim no)
+		(in_bom yes)
+		(on_board yes)
+		(in_pos_files yes)
+		(dnp no)
+		(property "Reference" "#FLG02"
+			(at 112.395 20.32 0)
+			(hide yes)
+			(show_name no)
+			(do_not_autoplace no)
+			(effects
+				(font
+					(size 1.27 1.27)
+				)
+			)
+		)
+		(property "Value" "PWR_FLAG"
+			(at 111.76 18.796 90)
+			(show_name no)
+			(do_not_autoplace no)
+			(effects
+				(font
+					(size 1.27 1.27)
+				)
+				(justify left)
+			)
+		)
+		(property "Footprint" ""
+			(at 114.3 20.32 0)
+			(hide yes)
+			(show_name no)
+			(do_not_autoplace no)
+			(effects
+				(font
+					(size 1.27 1.27)
+				)
+			)
+		)
+		(property "Datasheet" ""
+			(at 114.3 20.32 0)
+			(hide yes)
+			(show_name no)
+			(do_not_autoplace no)
+			(effects
+				(font
+					(size 1.27 1.27)
+				)
+			)
+		)
+		(property "Description" "Special symbol for telling ERC where power comes from"
+			(at 114.3 20.32 0)
+			(hide yes)
+			(show_name no)
+			(do_not_autoplace no)
+			(effects
+				(font
+					(size 1.27 1.27)
+				)
+			)
+		)
+		(pin "1"
+		)
+		(instances
+			(project "mother"
+				(path "/7a893922-4a26-4218-912f-8bb60bebfa2a"
+					(reference "#FLG02")
 					(unit 1)
 				)
@@
 			)
 		)
-		(property "Footprint" ""
+		(property "Footprint" "Connector_PinSocket_2.54mm:PinSocket_1x06_P2.54mm_Vertical"
 			(at 77.47 39.37 0)
 			(hide yes)

Commit message: push just to make sure everything is up to date
Parts:
- removed D102: SMAJ26A, Diode_SMD:D_SMA, symbol Diode:SMAJ26A
- added D102: SMAJ26CA, Diode_SMD:D_SMA, symbol Diode:SMAJ26CA
Connections:
- net GND: now also R101.2, D102.1 (A1); no longer D101.1 (K)
- net at C101.1, C102.1, C103.1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: now also D101.1 (K), D102.2 (A2); no longer R101.1
- net at D101.2 (A), Q101.1 (G): now also R101.1; no longer R101.2
Other:
- moved on the sheet: F101, J101, Q101

Commit message: WIP motherboard pcb save point, layout and partial routing complete
Connections:
- net Q101_Drain: now reaches C101.1, C102.1, C103.1, D101.1 (K), D102.2 (A2), Q101.3 (D), R102.2, R103.2
Other:
- moved on the sheet: D101

Commit message: finished pcb, updated schematic formatting, ready for fab
Other:
- note added: "5/3/2026"
- note added: "JFET Preamp with ADC Motherboard By Lucas Samaniego"
- moved on the sheet: C101, C102, C103, D101, D102, D103, F101, J101, J102, J103, Q101, R101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

Commit message: fixed TVS Diodes across 4 channels and redo placement and traces
Parts:
- C101, F101, J101, J102, J103: now left out of the parts list
- C102: LCSC Part # (none) -> C15849
- C103: LCSC Part # (none) -> C14663
- D101: LCSC Part # (none) -> C545374
- D102: LCSC Part # (none) -> C148226
- D103: LCSC Part # (none) -> C2286
- Q101: LCSC Part # (none) -> C15127
- R101: LCSC Part # (none) -> C25803
- R102: LCSC Part # (none) -> C21189
- R103: LCSC Part # (none) -> C25999
Changed lines of the file:
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@@
+			)
+		)
+		(property "LCSC Part #" "C545374"
+			(at 160.02 59.69 90)
+			(hide yes)
+			(show_name no)
+			(do_not_autoplace no)
+			(effects
+				(font
+					(size 1.27 1.27)
+				)
 			)
 		)
@@
 		(body_style 1)
 		(exclude_from_sim no)
-		(in_bom yes)
+		(in_bom no)
 		(on_board yes)
 		(in_pos_files yes)
@@
 			)
 		)
+		(property "LCSC Part #" ""
+			(at 175.26 55.88 90)
+			(hide yes)
+			(show_name no)
+			(do_not_autoplace no)
+			(effects
+				(font
+					(size 1.27 1.27)
+				)
+			)
+		)
 		(pin "1"
 		)
@@
 			)
 		)
+		(property "LCSC Part #" "C148226"
+			(at 140.97 60.96 90)
+			(hide yes)
+			(show_name no)
+			(do_not_autoplace no)
+			(effects
+				(font
+					(size 1.27 1.27)
+				)
+			)
+		)
 		(pin "1"
 		)
@@
 			)
 		)
+		(property "LCSC Part #" "C21189"
+			(at 116.84 50.8 0)
+			(hide yes)
+			(show_name no)
+			(do_not_autoplace no)
+			(effects
+				(font
+					(size 1.27 1.27)
+				)
+			)
+		)
 		(pin "2"
 		)
@@
 			)
 		)
+		(property "LCSC Part #" "C25803"
+			(at 165.1 68.58 0)
+			(hide yes)
+			(show_name no)
+			(do_not_autoplace no)
+			(effects
+				(font
+					(size 1.27 1.27)
+				)
+			)
+		)
 		(pin "1"
 		)
@@
 		(property "Description" "Resistor"
 			(at 106.68 55.88 0)
+			(hide yes)
+			(show_name no)
+			(do_not_autoplace no)
+			(effects
+				(font
+					(size 1.27 1.27)
+				)
+			)
+		)
+		(property "LCSC Part #" "C25999"
+			(at 106.68 55.88 90)
 			(hide yes)
 			(show_name no)
@@
 			)
 		)
+		(property "LCSC Part #" "C15127"
+			(at 165.1 58.42 90)
+			(hide yes)
+			(show_name no)
+			(do_not_autoplace no)
+			(effects
+				(font
+					(size 1.27 1.27)
+				)
+			)
+		)
 		(pin "1"
 		)
@@
 		(body_style 1)
 		(exclude_from_sim no)
-		(in_bom yes)
+		(in_bom no)
 		(on_board yes)
 		(in_pos_files yes)
@@
 			)
 		)
+		(property "LCSC Part #" ""
+			(at 132.08 60.96 0)
+			(hide yes)
+			(show_name no)
+			(do_not_autoplace no)
+			(effects
+				(font
+					(size 1.27 1.27)
+				)
+			)
+		)
 		(pin "1"
 		)
@@
 		(body_style 1)
 		(exclude_from_sim no)
-		(in_bom yes)
+		(in_bom no)
 		(on_board yes)
 		(in_pos_files yes)
@@
 			)
 		)
+		(property "LCSC Part #" ""
+			(at 76.2 66.04 90)
+			(hide yes)
+			(show_name no)
+			(do_not_autoplace no)
+			(effects
+				(font
+					(size 1.27 1.27)
+				)
+			)
+		)
 		(pin "2"
 		)
@@
 			)
 		)
+		(property "LCSC Part #" "C15849"
+			(at 121.92 60.96 0)
+			(hide yes)
+			(show_name no)
+			(do_not_autoplace no)
+			(effects
+				(font
+					(size 1.27 1.27)
+				)
+			)
+		)
 		(pin "1"
 		)
@@
 			)
 		)
+		(property "LCSC Part #" "C2286"
+			(at 102.87 62.23 90)
+			(hide yes)
+			(show_name no)
+			(do_not_autoplace no)
+			(effects
+				(font
+					(size 1.27 1.27)
+				)
+			)
+		)
 		(pin "1"
 		)
@@
 			)
 		)
+		(property "LCSC Part #" "C14663"
+			(at 111.76 60.96 0)
+			(hide yes)
+			(show_name no)
+			(do_not_autoplace no)
+			(effects
+				(font
+					(size 1.27 1.27)
+				)
+			)
+		)
 		(pin "1"
 		)
@@
 		(body_style 1)
 		(exclude_from_sim no)
-		(in_bom yes)
+		(in_bom no)
 		(on_board yes)
 		(in_pos_files yes)
@@
 			)
 		)
+		(property "LCSC Part #" ""
+			(at 186.69 55.88 0)
+			(hide yes)
+			(show_name no)
+			(do_not_autoplace no)
+			(effects
+				(font
+					(size 1.27 1.27)
+				)
+			)
+		)
 		(pin "1"
 		)
@@
 		(body_style 1)
 		(exclude_from_sim no)
-		(in_bom yes)
+		(in_bom no)
 		(on_board yes)
 		(in_pos_files yes)
@@
 			(hide yes)
 			(show_name no)
+			(do_not_autoplace no)
+			(effects
+				(font
+					(size 1.27 1.27)
+				)
+			)
+		)
+		(property "LCSC Part #" ""
+			(at 78.74 52.07 90)
+			(hide yes)
+			(show_name no)
