File: JFET_Preamp_Mother/preamp_channel.kicad_sch (KiCad schematic)
At the start: 19 parts, among them J201 XLR3, Q201 2SK209, Q202 2SK209, Q203 2SK209

Commit message: motherboard .sch erc clean
Parts:
- D201, D202: footprint MMBZ27VALT1G:SOT95P237X111-3N -> Package_TO_SOT_SMD:SOT-23
Changed lines of the file:
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@@
 			)
 		)
-		(property "Footprint" "MMBZ27VALT1G:SOT95P237X111-3N"
+		(property "Footprint" "Package_TO_SOT_SMD:SOT-23"
 			(at 97.79 86.36 0)
 			(hide yes)
@@
 			)
 		)
-		(property "Footprint" "MMBZ27VALT1G:SOT95P237X111-3N"
+		(property "Footprint" "Package_TO_SOT_SMD:SOT-23"
 			(at 102.87 64.77 0)
 			(hide yes)

Commit message: finish draft of mother/daughter sch and start routing, reconcile libraries and missing footprints
Parts:
- added R211, R212, R213: 0, Resistor_SMD:R_0603_1608Metric, symbol Device:R
- renumbered R215 to R209, R219 to R210
Connections:
- net CH_GND: now also R213.2; no longer J201.1
- net D_TVS_COLD: now also R211.1; no longer C203.2, D202.2 (A2), R202.2
- net D_TVS_HOT: now also R212.2; no longer J201.2
- new net: C203.2, D202.2 (A2), R202.2, R211.2
- new net: J201.1, R213.1
- new net: J201.2, R212.1
Other:
- moved on the sheet: C201, C202, C203, D201, D202, J201, Q201, Q202, Q203, R201, R202, R203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

Commit message: finished pcb, updated schematic formatting, ready for fab
Other:
- note added: "5/3/2026"
- note added: "JFET Preamp Channel By Lucas Samaniego"
Changed lines of the file:
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@@
 	(generator_version "10.0")
 	(paper "A5")
+	(text "5/3/2026\n"
+		(exclude_from_sim no)
+		(at 124.46 131.318 0)
+		(effects
+			(font
+				(size 1.27 1.27)
+			)
+		)
+	)
+	(text "JFET Preamp Channel				By Lucas Samaniego"
+		(exclude_from_sim no)
+		(at 129.794 127.762 0)
+		(effects
+			(font
+				(size 1.27 1.27)
+			)
+		)
+	)
 	(junction
 		(at 129.54 53.34)

Commit message: fixed TVS Diodes across 4 channels and redo placement and traces
Parts:
- C201, C202, C203: LCSC Part # (none) -> C1603
- D201, D202: footprint Package_TO_SOT_SMD:SOT-23 -> Diode_SMD:D_SMA; LCSC Part # (none) -> C148226
- J201: now left out of the parts list
- Q201, Q202, Q203: LCSC Part # (none) -> C2880444
- R201, R202, R205, R209: LCSC Part # (none) -> C137687
- R203, R204, R208, R210: LCSC Part # (none) -> C23156
- R206: LCSC Part # (none) -> C25117
- R207: LCSC Part # (none) -> C22808
- R211, R212, R213: LCSC Part # (none) -> C21189
